Commit message: Add MoveIt configuration package for grinding robot with various planning settings

File: onolab_ws/src/grinding_robot_description/urdf/ur5e_with_pestle.urdf.xacro (robot description, xacro)
@@ -1,46 +1,105 @@
 <?xml version="1.0"?>
 <robot xmlns:xacro="http://wiki.ros.org/xacro" name="$(arg name)">
-   <!-- robot name parameter -->
-   <xacro:arg name="name" default="ur"/>
-   <!-- import main macro -->
-   <xacro:include filename="$(find ur_description)/urdf/ur_macro.xacro"/>
-   <!-- possible 'ur_type' values: ur3, ur3e, ur5, ur5e, ur10, ur10e, ur16e, ur20, ur30 -->
-   <!-- the default value should raise an error in case this was called without defining the type -->
-   <xacro:arg name="ur_type" default="ur5e"/>
-   <!-- parameters -->
-   <xacro:arg name="tf_prefix" default="" />
-   <xacro:arg name="joint_limit_params" default="$(find ur_description)/config/$(arg ur_type)/joint_limits.yaml"/>
-   <xacro:arg name="kinematics_params" default="$(find ur_description)/config/$(arg ur_type)/default_kinematics.yaml"/>
-   <xacro:arg name="physical_params" default="$(find ur_description)/config/$(arg ur_type)/physical_parameters.yaml"/>
-   <xacro:arg name="visual_params" default="$(find ur_description)/config/$(arg ur_type)/visual_parameters.yaml"/>
-   <xacro:arg name="transmission_hw_interface" default=""/>
-   <xacro:arg name="safety_limits" default="false"/>
-   <xacro:arg name="safety_pos_margin" default="0.15"/>
-   <xacro:arg name="safety_k_position" default="20"/>
-   <xacro:arg name="pestle_length" default="0.12" />
-   <xacro:arg name="spatula_length" default="0.089" />
-   <!--When using gazebo simulations absolute paths are necessary.-->
-   <xacro:arg name="force_abs_paths" default="false" />
-   <!-- create link fixed to the "world" -->
-   <link name="world" />
-   <!-- arm -->
-   <xacro:ur_robot
-     name="$(arg name)"
-     tf_prefix="$(arg tf_prefix)"
-     parent="world"
-     joint_limits_parameters_file="$(arg joint_limit_params)"
-     kinematics_parameters_file="$(arg kinematics_params)"
-     physical_parameters_file="$(arg physical_params)"
-     visual_parameters_file="$(arg visual_params)"
-     safety_limits="$(arg safety_limits)"
-     safety_pos_margin="$(arg safety_pos_margin)"
-     safety_k_position="$(arg safety_k_position)"
-     force_abs_paths="$(arg force_abs_paths)"
-     >
-     <origin xyz="0 0 0" rpy="0 0 0" />          <!-- position robot in the world -->
-   </xacro:ur_robot>
-   <!-- Add end effector frames -->
-    <xacro:property name="pestle_mesh" value="$(find grinding_robot_description)/meshes/end_effector/pestle_ur.stl"/>
-    <xacro:property name="spatula_mesh" value="$(find grinding_robot_description)/meshes/end_effector/spatula.stl"/>
+    <!-- robot name parameter -->
+    <xacro:arg name="name" default="ur" />
+    <xacro:include filename="$(find ur_description)/urdf/ur_macro.xacro" />
+    <!-- ros2 control include -->
+    <xacro:include filename="$(find ur_robot_driver)/urdf/ur.ros2_control.xacro" />
+    <xacro:include filename="$(find ur_description)/urdf/inc/ur_transmissions.xacro" />
+    <!-- possible 'ur_type' values: ur3, ur3e, ur5, ur5e, ur10, ur10e, ur16e, ur20 -->
+    <!-- the default value should raise an error in case this was called without defining the type -->
+    <xacro:arg name="ur_type" default="urXe" />
+    <!-- parameters -->
+    <xacro:arg name="tf_prefix" default="" />
+    <xacro:arg name="joint_limit_params"
+        default="$(find ur_description)/config/$(arg ur_type)/joint_limits.yaml" />
+    <xacro:arg name="kinematics_params"
+        default="$(find ur_description)/config/$(arg ur_type)/default_kinematics.yaml" />
+    <xacro:arg name="physical_params"
+        default="$(find ur_description)/config/$(arg ur_type)/physical_parameters.yaml" />
+    <xacro:arg name="visual_params"
+        default="$(find ur_description)/config/$(arg ur_type)/visual_parameters.yaml" />
+    <xacro:arg name="transmission_hw_interface" default="" />
+    <xacro:arg name="safety_limits" default="false" />
+    <xacro:arg name="safety_pos_margin" default="0.15" />
+    <xacro:arg name="safety_k_position" default="20" />
+    <!-- ros2_control related parameters -->
+    <xacro:arg name="headless_mode" default="false" />
+    <xacro:arg name="robot_ip" default="0.0.0.0" />
+    <xacro:arg name="script_filename" default="" />
+    <xacro:arg name="output_recipe_filename" default="" />
+    <xacro:arg name="input_recipe_filename" default="" />
+    <xacro:arg name="reverse_ip" default="0.0.0.0" />
+    <xacro:arg name="script_command_port" default="50004" />
+    <xacro:arg name="reverse_port" default="50001" />
+    <xacro:arg name="script_sender_port" default="50002" />
+    <xacro:arg name="trajectory_port" default="50003" />
+    <!--   tool communication related parameters-->
+    <xacro:arg name="use_tool_communication" default="false" />
+    <xacro:arg name="tool_voltage" default="0" />
+    <xacro:arg name="tool_parity" default="0" />
+    <xacro:arg name="tool_baud_rate" default="115200" />
+    <xacro:arg name="tool_stop_bits" default="1" />
+    <xacro:arg name="tool_rx_idle_chars" default="1.5" />
+    <xacro:arg name="tool_tx_idle_chars" default="3.5" />
+    <xacro:arg name="tool_device_name" default="/tmp/ttyUR" />
+    <xacro:arg name="tool_tcp_port" default="54321" />
+    <!-- Simulation parameters -->
+    <xacro:arg name="use_mock_hardware" default="false" />
+    <xacro:arg name="mock_sensor_commands" default="false" />
+    <xacro:arg name="simulation_controllers" default="" />
+    <!-- initial position for simulations (Mock Hardware, Gazebo, Ignition) -->
+    <xacro:arg name="initial_positions_file"
+        default="$(find ur_description)/config/initial_positions.yaml" />
+    <!-- convert to property to use substitution in function -->
+    <xacro:property name="initial_positions_file" default="$(arg initial_positions_file)" />
+    <!-- create link fixed to the "world" -->
+    <link name="world" />
+    <xacro:ur_robot
+        name="$(arg name)"
+        tf_prefix="$(arg tf_prefix)"
+        parent="world"
+        joint_limits_parameters_file="$(arg joint_limit_params)"
+        kinematics_parameters_file="$(arg kinematics_params)"
+        physical_parameters_file="$(arg physical_params)"
+        visual_parameters_file="$(arg visual_params)"
+        safety_limits="$(arg safety_limits)"
+        safety_pos_margin="$(arg safety_pos_margin)"
+        safety_k_position="$(arg safety_k_position)"
+    >
+        <origin xyz="0 0 0" rpy="0 0 0" />          <!-- position robot in the world -->
+    </xacro:ur_robot>
+    <!-- ros2 control instance -->
+    <xacro:ur_ros2_control
+        name="$(arg name)"
+        tf_prefix="$(arg tf_prefix)"
+        kinematics_parameters_file="$(arg kinematics_params)"
+        transmission_hw_interface="$(arg transmission_hw_interface)"
+        use_mock_hardware="$(arg use_mock_hardware)"
+        mock_sensor_commands="$(arg mock_sensor_commands)"
+        headless_mode="$(arg headless_mode)"
+        initial_positions="${xacro.load_yaml(initial_positions_file)}"
+        use_tool_communication="$(arg use_tool_communication)"
+        tool_voltage="$(arg tool_voltage)"
+        tool_parity="$(arg tool_parity)"
+        tool_baud_rate="$(arg tool_baud_rate)"
+        tool_stop_bits="$(arg tool_stop_bits)"
+        tool_rx_idle_chars="$(arg tool_rx_idle_chars)"
+        tool_tx_idle_chars="$(arg tool_tx_idle_chars)"
+        tool_device_name="$(arg tool_device_name)"
+        tool_tcp_port="$(arg tool_tcp_port)"
+        robot_ip="$(arg robot_ip)"
+        script_filename="$(arg script_filename)"
+        output_recipe_filename="$(arg output_recipe_filename)"
+        input_recipe_filename="$(arg input_recipe_filename)"
+        reverse_ip="$(arg reverse_ip)"
+        script_command_port="$(arg script_command_port)"
+        reverse_port="$(arg reverse_port)"
+        script_sender_port="$(arg script_sender_port)"
+        trajectory_port="$(arg trajectory_port)"
+    />
+    <!-- Add end effector frames -->
+    <xacro:arg name="pestle_length" default="0.12" />
+    <xacro:arg name="spatula_length" default="0.089" />
     <xacro:macro name="end_effectors" params="prefix pestle_length spatula_length">
         <!-- Default tool frames -->
@@ -68,5 +127,6 @@
                 <origin xyz="0 0 0.0001" rpy="0 0 0" />
                 <geometry>
-                    <mesh filename="package://grinding_robot_description/meshes/end_effector/pestle_ur.stl" />
+                    <mesh
+                        filename="package://grinding_robot_description/meshes/end_effector/pestle_ur.stl" />
                 </geometry>
             </visual>
@@ -88,5 +148,6 @@
                 <origin xyz="0 0 0.0001" rpy="0 0 0" />
                 <geometry>
-                    <mesh filename="package://grinding_robot_description/meshes/end_effector/spatula.stl" />
+                    <mesh
+                        filename="package://grinding_robot_description/meshes/end_effector/spatula.stl" />
                 </geometry>
             </visual>
@@ -111,4 +172,5 @@
         </joint>
     </xacro:macro>
-    <xacro:end_effectors prefix="$(arg tf_prefix)" pestle_length="$(arg pestle_length)" spatula_length="$(arg spatula_length)" />
+    <xacro:end_effectors prefix="$(arg tf_prefix)" pestle_length="$(arg pestle_length)"
+        spatula_length="$(arg spatula_length)" />
 </robot>
